Commit message: tess setup

File: urdf/combined.urdf (robot description, URDF)
Before this commit: robot combined, 33 links, 32 joints
Links:
- link ABB1200_base_link: geometry collision mesh filename=model://abb/meshes/collision/base_link.stl scale=1 1 1; visual mesh filename=model://abb/meshes/visual/base_link.dae scale=1 1 1
- link ABB1200_link_1: geometry collision mesh filename=model://abb/meshes/collision/link_1.stl scale=1 1 1; visual mesh filename=model://abb/meshes/visual/link_1.dae scale=1 1 1
- link ABB1200_link_2: geometry collision mesh filename=model://abb/meshes/collision/link_2.stl scale=1 1 1; visual mesh filename=model://abb/meshes/visual/link_2.dae scale=1 1 1
- link ABB1200_link_3: geometry collision mesh filename=model://abb/meshes/collision/link_3.stl scale=1 1 1; visual mesh filename=model://abb/meshes/visual/link_3.dae scale=1 1 1
- link ABB1200_link_4: geometry collision mesh filename=model://abb/meshes/collision/link_4.stl scale=1 1 1; visual mesh filename=model://abb/meshes/visual/link_4.dae scale=1 1 1
- link ABB1200_link_5: geometry collision mesh filename=model://abb/meshes/collision/link_5.stl scale=1 1 1; visual mesh filename=model://abb/meshes/visual/link_5.dae scale=1 1 1
- link ABB1200_link_6: geometry collision mesh filename=model://abb/meshes/collision/link_6.stl scale=1 1 1; visual mesh filename=model://abb/meshes/visual/link_6.dae scale=1 1 1

Commit message: distance check test

File: urdf/combined.urdf (robot description, URDF)
Before this commit: robot combined, 33 links, 32 joints
Links:
- link ABB1200_base_link: geometry visual mesh filename=model://abb/meshes/visual/base_link.dae scale=1 1 1
- link controller_box: geometry 
- link right_arm_base_link: geometry visual mesh filename=model://sawyer/meshes/sawyer_pv/base.DAE

Commit message: tess working

File: urdf/combined.urdf (robot description, URDF)
Before this commit: robot combined, 33 links, 32 joints
Joints:
- joint sawyer_pose: origin xyz=0. 0. 0.11 rpy=0 0 0 -> xyz=0. 0. 0.93 rpy=0 0 0
